File: pcb/esp-thermostat/_autosave-esp-thermostat.kicad_pcb (KiCad board)
At the start: 2 copper layers, 87 x 87 mm, 56 parts, among them J1 AC IN, J2 RELAY, J3 OLED, J4 PROGRAM, J5 DS18B20+, K1 HK4100F-DC5V-SHG, Q1 SS8050-G, Q2 SS8050-G, Q3 AO3480, SW1 SW_PLUS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

Commit message: PCB: add temp sensor header, optimize routing
Parts:
- BT1: value Battery_Cell -> 3V CR1632
- U3: value 47L04 -> 47L16
Routing:
- net +3V3: track 224.8 -> 235.1 mm
- net ESP_~RST~: track 28.2 -> 28.8 mm, vias 3 -> 2
- net GND: vias 37 -> 38
Changed lines of the file:
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@@
     (thickness 1.6)
     (drawings 36)
-    (tracks 542)
+    (tracks 546)
     (zones 0)
     (modules 56)
@@
   )
   (setup
-    (last_trace_width 0.3048)
+    (last_trace_width 0.4064)
     (user_trace_width 0.3048)
     (user_trace_width 0.4064)
@@
       (effects (font (size 1 1) (thickness 0.15)))
     )
-    (fp_text value Battery_Cell (at 0 -6.85 180) (layer F.Fab)
+    (fp_text value "3V CR1632" (at 0 -6.85 180) (layer F.Fab)
       (effects (font (size 1 1) (thickness 0.15)))
     )
@@
       (effects (font (size 1 1) (thickness 0.15)))
     )
-    (fp_text value 47L04 (at 0 3.4 90) (layer F.Fab)
+    (fp_text value 47L16 (at 0 3.4 90) (layer F.Fab)
       (effects (font (size 1 1) (thickness 0.15)))
     )
@@
   (via (at 45.2 97.9) (size 0.5) (drill 0.3) (layers F.Cu B.Cu) (net 21))
   (via (at 45.1 99.5) (size 0.5) (drill 0.3) (layers F.Cu B.Cu) (net 21))
+  (via (at 43.2 98.3) (size 0.5) (drill 0.3) (layers F.Cu B.Cu) (net 21))
   (segment (start 36.154998 71.1) (end 35.554999 70.500001) (width 0.4064) (layer F.Cu) (net 22))
   (segment (start 37.55 71.1) (end 36.154998 71.1) (width 0.4064) (layer F.Cu) (net 22))
@@
   (segment (start 46.25 95.35) (end 46.2 95.3) (width 0.8128) (layer F.Cu) (net 22))
   (segment (start 46.25 100.875) (end 46.25 95.35) (width 0.8128) (layer F.Cu) (net 22))
+  (segment (start 35.054 101.625) (end 35.079 101.6) (width 0.4064) (layer F.Cu) (net 22))
+  (segment (start 34.254 101.625) (end 35.054 101.625) (width 0.4064) (layer F.Cu) (net 22))
+  (segment (start 35.079 101.6) (end 42 101.6) (width 0.4064) (layer F.Cu) (net 22))
+  (segment (start 42.725 100.875) (end 44.25 100.875) (width 0.4064) (layer F.Cu) (net 22))
+  (segment (start 42 101.6) (end 42.725 100.875) (width 0.4064) (layer F.Cu) (net 22))
   (via (at 44.2 83.1) (size 0.5) (drill 0.3) (layers F.Cu B.Cu) (net 23))
   (segment (start 44.2 84.275) (end 44.2 83.1) (width 0.3048) (layer B.Cu) (net 23))
@@
   (segment (start 53.45 93.9) (end 52.4 93.9) (width 0.3048) (layer F.Cu) (net 27))
   (segment (start 52.4 93.9) (end 51.9 94.4) (width 0.3048) (layer F.Cu) (net 27))
-  (via (at 35.7 100) (size 0.5) (drill 0.3) (layers F.Cu B.Cu) (net 27))
-  (segment (start 35.702401 99.997599) (end 35.7 100) (width 0.3048) (layer B.Cu) (net 27))
   (segment (start 34.679 100) (end 34.254 99.575) (width 0.3048) (layer F.Cu) (net 27))
-  (segment (start 35.7 100) (end 34.679 100) (width 0.3048) (layer F.Cu) (net 27))
   (segment (start 51.9 94.4) (end 48.2 98.1) (width 0.3048) (layer B.Cu) (net 27))
-  (segment (start 41.6 100) (end 35.7 100) (width 0.3048) (layer F.Cu) (net 27))
   (segment (start 48.2 98.1) (end 47.7 98.6) (width 0.3048) (layer B.Cu) (net 27))
   (segment (start 47.7 98.6) (end 47.6 98.7) (width 0.3048) (layer B.Cu) (net 27))
   (via (at 45.1 98.7) (size 0.5) (drill 0.3) (layers F.Cu B.Cu) (net 27))
   (segment (start 47.6 98.7) (end 45.1 98.7) (width 0.3048) (layer B.Cu) (net 27))
-  (segment (start 42.1 100) (end 41.6 100) (width 0.3048) (layer F.Cu) (net 27))
-  (segment (start 44.746447 98.7) (end 44.346447 99.1) (width 0.3048) (layer F.Cu) (net 27))
-  (segment (start 45.1 98.7) (end 44.746447 98.7) (width 0.3048) (layer F.Cu) (net 27))
-  (segment (start 43 99.1) (end 42.1 100) (width 0.3048) (layer F.Cu) (net 27))
-  (segment (start 44.346447 99.1) (end 43 99.1) (width 0.3048) (layer F.Cu) (net 27))
+  (segment (start 34.675 99.575) (end 35.1 100) (width 0.3048) (layer F.Cu) (net 27))
+  (segment (start 34.254 99.575) (end 34.675 99.575) (width 0.3048) (layer F.Cu) (net 27))
+  (segment (start 35.1 100) (end 42.1 100) (width 0.3048) (layer F.Cu) (net 27))
+  (segment (start 42.1 100) (end 43 99.1) (width 0.3048) (layer F.Cu) (net 27))
+  (segment (start 43 99.1) (end 44.346447 99.1) (width 0.3048) (layer F.Cu) (net 27))
+  (segment (start 44.746447 98.7) (end 45.1 98.7) (width 0.3048) (layer F.Cu) (net 27))
+  (segment (start 44.346447 99.1) (end 44.746447 98.7) (width 0.3048) (layer F.Cu) (net 27))
   (segment (start 36.2 93.6) (end 36.2 95.3) (width 0.3048) (layer F.Cu) (net 28))
   (segment (start 36.2 92.225) (end 36.2 93.6) (width 0.3048) (layer B.Cu) (net 28))
