File: pcb/esp-thermostat/esp-thermostat.sch (KiCad schematic (older format))
At the start: 30 parts, among them J1 AC IN, J2 RELAY, J3 OLED, J4 PROGRAM, K1 HK4100F-DC5V-SHG, Q1 SS8050-G, Q2 SS8050-G, Q3 AO3480, SW1 SW_PLUS, SW2 SW_BOOST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

Commit message: PCB: add temp sensor header, optimize routing
Parts:
- added J5: DS18B20+, Connector_PinHeader_2.54mm:PinHeader_1x03_P2.54mm_Vertical, symbol w_connectors:HEADER_3
Connections:
- net +3V3: now also J5.1
- net GND: now also J5.3
- new net ESP_1W_DQ: J5.2
Changed lines of the file:
@@
 EESchema Schematic File Version 4
+LIBS:esp-thermostat-cache
 EELAYER 30 0
 EELAYER END
@@
 	1    0    0    -1
 $EndComp
+$Comp
+L w_connectors:HEADER_3 J?
+U 1 1 5E092C8B
+P 3300 3800
+AR Path="/5DE7044F/5E092C8B" Ref="J?"  Part="1"
+AR Path="/5E092C8B" Ref="J5"  Part="1"
+F 0 "J5" H 3428 3853 60  0000 L CNN
+F 1 "DS18B20+" H 3428 3747 60  0000 L CNN
+F 2 "Connector_PinHeader_2.54mm:PinHeader_1x03_P2.54mm_Vertical" H 3300 3800 60  0001 C CNN
+F 3 "" H 3300 3800 60  0000 C CNN
+	1    3300 3800
+	1    0    0    -1
+$EndComp
+Wire Wire Line
+	3200 3700 3100 3700
+Wire Wire Line
+	3100 3700 3100 3600
+Wire Wire Line
+	3200 3900 3100 3900
+Wire Wire Line
+	3100 3900 3100 4000
+Wire Wire Line
+	3200 3800 3100 3800
+Text GLabel 3100 3800 0    50   BiDi ~ 0
+ESP_1W_DQ
+$Comp
+L power:GND #PWR?
+U 1 1 5E092C97
+P 3100 4000
+AR Path="/5DE7044F/5E092C97" Ref="#PWR?"  Part="1"
+AR Path="/5E092C97" Ref="#PWR0137"  Part="1"
+F 0 "#PWR0137" H 3100 3750 50  0001 C CNN
+F 1 "GND" H 3105 3827 50  0000 C CNN
+F 2 "" H 3100 4000 50  0001 C CNN
+F 3 "" H 3100 4000 50  0001 C CNN
+	1    3100 4000
+	1    0    0    -1
+$EndComp
+$Comp
+L power:+3.3V #PWR?
+U 1 1 5E092C9D
+P 3100 3600
+AR Path="/5DE7044F/5E092C9D" Ref="#PWR?"  Part="1"
+AR Path="/5E092C9D" Ref="#PWR0138"  Part="1"
+F 0 "#PWR0138" H 3100 3450 50  0001 C CNN
+F 1 "+3.3V" H 3115 3773 50  0000 C CNN
+F 2 "" H 3100 3600 50  0001 C CNN
+F 3 "" H 3100 3600 50  0001 C CNN
+	1    3100 3600
+	1    0    0    -1
+$EndComp

Commit message: PCB: prepare for manufacturing
Parts:
- added C10, C11: 100n, Capacitor_SMD:C_0805_2012Metric_Pad1.15x1.40mm_HandSolder, symbol Device:C
- added C9: 1000u, Capacitor_THT:CP_Radial_D10.0mm_P5.00mm, symbol Device:CP
- H1, H2, H3, H4, H5: footprint MountingHole:MountingHole_2.2mm_M2_ISO14580_Pad -> MountingHole:MountingHole_3.2mm_M3_ISO14580_Pad
Connections:
- net +3V3: now also C10.1, C11.1, C9.1
- net GND: now also C10.2, C11.2, C9.2
Changed lines of the file:
@@
 L power:+3.3V #PWR0126
 U 1 1 5DDA81B3
-P 1600 4750
-F 0 "#PWR0126" H 1600 4600 50  0001 C CNN
-F 1 "+3.3V" H 1615 4923 50  0000 C CNN
-F 2 "" H 1600 4750 50  0001 C CNN
-F 3 "" H 1600 4750 50  0001 C CNN
-	1    1600 4750
+P 1600 4700
+F 0 "#PWR0126" H 1600 4550 50  0001 C CNN
+F 1 "+3.3V" H 1615 4873 50  0000 C CNN
+F 2 "" H 1600 4700 50  0001 C CNN
+F 3 "" H 1600 4700 50  0001 C CNN
+	1    1600 4700
 	1    0    0    -1
 $EndComp
@@
 L power:GND #PWR0127
 U 1 1 5DDA8F74
-P 1600 5250
-F 0 "#PWR0127" H 1600 5000 50  0001 C CNN
-F 1 "GND" H 1605 5077 50  0000 C CNN
-F 2 "" H 1600 5250 50  0001 C CNN
-F 3 "" H 1600 5250 50  0001 C CNN
-	1    1600 5250
+P 1600 5300
+F 0 "#PWR0127" H 1600 5050 50  0001 C CNN
+F 1 "GND" H 1605 5127 50  0000 C CNN
+F 2 "" H 1600 5300 50  0001 C CNN
+F 3 "" H 1600 5300 50  0001 C CNN
+	1    1600 5300
 	1    0    0    -1
 $EndComp
@@
 	1700 4850 1600 4850
 Wire Wire Line
-	1600 4850 1600 4750
-Wire Wire Line
 	1700 4950 1600 4950
-Wire Wire Line
-	1600 4950 1600 5250
 Wire Wire Line
 	1700 5050 1500 5050
@@
 F 0 "H1" H 1050 1846 50  0000 L CNN
 F 1 "MountingHole" H 1050 1755 50  0000 L CNN
-F 2 "MountingHole:MountingHole_2.2mm_M2_ISO14580_Pad" H 950 1800 50  0001 C CNN
+F 2 "MountingHole:MountingHole_3.2mm_M3_ISO14580_Pad" H 950 1800 50  0001 C CNN
 F 3 "~" H 950 1800 50  0001 C CNN
 	1    950  1800
@@
 F 0 "H2" H 1050 2046 50  0000 L CNN
 F 1 "MountingHole" H 1050 1955 50  0000 L CNN
-F 2 "MountingHole:MountingHole_2.2mm_M2_ISO14580_Pad" H 950 2000 50  0001 C CNN
+F 2 "MountingHole:MountingHole_3.2mm_M3_ISO14580_Pad" H 950 2000 50  0001 C CNN
 F 3 "~" H 950 2000 50  0001 C CNN
 	1    950  2000
@@
 F 0 "H3" H 1050 2246 50  0000 L CNN
 F 1 "MountingHole" H 1050 2155 50  0000 L CNN
-F 2 "MountingHole:MountingHole_2.2mm_M2_ISO14580_Pad" H 950 2200 50  0001 C CNN
+F 2 "MountingHole:MountingHole_3.2mm_M3_ISO14580_Pad" H 950 2200 50  0001 C CNN
 F 3 "~" H 950 2200 50  0001 C CNN
 	1    950  2200
@@
 F 0 "H4" H 1050 2446 50  0000 L CNN
 F 1 "MountingHole" H 1050 2355 50  0000 L CNN
-F 2 "MountingHole:MountingHole_2.2mm_M2_ISO14580_Pad" H 950 2400 50  0001 C CNN
+F 2 "MountingHole:MountingHole_3.2mm_M3_ISO14580_Pad" H 950 2400 50  0001 C CNN
 F 3 "~" H 950 2400 50  0001 C CNN
 	1    950  2400
 	1    0    0    -1
 $EndComp
-Wire Wire Line
-	8000 5700 8300 5700
 Wire Wire Line
 	8300 5500 8250 5500
@@
 F 0 "H5" H 1050 2646 50  0000 L CNN
 F 1 "MountingHole" H 1050 2555 50  0000 L CNN
-F 2 "MountingHole:MountingHole_2.2mm_M2_ISO14580_Pad" H 950 2600 50  0001 C CNN
+F 2 "MountingHole:MountingHole_3.2mm_M3_ISO14580_Pad" H 950 2600 50  0001 C CNN
 F 3 "~" H 950 2600 50  0001 C CNN
 	1    950  2600
@@
 	3200 3700 3100 3700
 Wire Wire Line
-	3100 3700 3100 3600
-Wire Wire Line
 	3200 3900 3100 3900
-Wire Wire Line
-	3100 3900 3100 4000
 Wire Wire Line
 	3200 3800 3100 3800
@@
 L power:GND #PWR?
 U 1 1 5E092C97
-P 3100 4000
+P 3100 4050
 AR Path="/5DE7044F/5E092C97" Ref="#PWR?"  Part="1"
 AR Path="/5E092C97" Ref="#PWR0137"  Part="1"
-F 0 "#PWR0137" H 3100 3750 50  0001 C CNN
-F 1 "GND" H 3105 3827 50  0000 C CNN
-F 2 "" H 3100 4000 50  0001 C CNN
-F 3 "" H 3100 4000 50  0001 C CNN
-	1    3100 4000
+F 0 "#PWR0137" H 3100 3800 50  0001 C CNN
+F 1 "GND" H 3105 3877 50  0000 C CNN
+F 2 "" H 3100 4050 50  0001 C CNN
+F 3 "" H 3100 4050 50  0001 C CNN
+	1    3100 4050
 	1    0    0    -1
 $EndComp
@@
 L power:+3.3V #PWR?
 U 1 1 5E092C9D
-P 3100 3600
+P 3100 3550
 AR Path="/5DE7044F/5E092C9D" Ref="#PWR?"  Part="1"
 AR Path="/5E092C9D" Ref="#PWR0138"  Part="1"
-F 0 "#PWR0138" H 3100 3450 50  0001 C CNN
-F 1 "+3.3V" H 3115 3773 50  0000 C CNN
-F 2 "" H 3100 3600 50  0001 C CNN
-F 3 "" H 3100 3600 50  0001 C CNN
-	1    3100 3600
-	1    0    0    -1
-$EndComp
+F 0 "#PWR0138" H 3100 3400 50  0001 C CNN
+F 1 "+3.3V" H 3115 3723 50  0000 C CNN
+F 2 "" H 3100 3550 50  0001 C CNN
+F 3 "" H 3100 3550 50  0001 C CNN
+	1    3100 3550
+	1    0    0    -1
+$EndComp
+Wire Wire Line
+	8000 5700 8300 5700
+$Comp
+L Device:CP C9
+U 1 1 5E140B19
+P 5000 950
+F 0 "C9" H 5118 996 50  0000 L CNN
+F 1 "1000u" H 5118 905 50  0000 L CNN
+F 2 "Capacitor_THT:CP_Radial_D10.0mm_P5.00mm" H 5038 800 50  0001 C CNN
+F 3 "~" H 5000 950 50  0001 C CNN
+	1    5000 950
+	1    0    0    -1
+$EndComp
+Wire Wire Line
+	4500 750  5000 750
+Wire Wire Line
+	5000 750  5000 800
+Wire Wire Line
+	4500 1150 5000 1150
+Wire Wire Line
+	5000 1150 5000 1100
+Wire Wire Line
+	1600 4950 1600 5250
+Wire Wire Line
+	1600 4700 1600 4750
+$Comp
+L Device:C C10
+U 1 1 5E166F79
+P 2350 5000
+F 0 "C10" H 2465 5046 50  0000 L CNN
+F 1 "100n" H 2465 4955 50  0000 L CNN
+F 2 "Capacitor_SMD:C_0805_2012Metric_Pad1.15x1.40mm_HandSolder" H 2388 4850 50  0001 C CNN
+F 3 "~" H 2350 5000 50  0001 C CNN
+	1    2350 5000
+	1    0    0    -1
+$EndComp
+$Comp
+L Device:C C11
+U 1 1 5E167B53
+P 4100 3800
+F 0 "C11" H 4215 3846 50  0000 L CNN
+F 1 "100n" H 4215 3755 50  0000 L CNN
+F 2 "Capacitor_SMD:C_0805_2012Metric_Pad1.15x1.40mm_HandSolder" H 4138 3650 50  0001 C CNN
+F 3 "~" H 4100 3800 50  0001 C CNN
+	1    4100 3800
+	1    0    0    -1
+$EndComp
+Wire Wire Line
+	1600 4750 2350 4750
+Wire Wire Line
+	2350 4750 2350 4850
+Connection ~ 1600 4750
+Wire Wire Line
+	1600 4750 1600 4850
+Wire Wire Line
+	2350 5150 2350 5250
+Wire Wire Line
+	2350 5250 1600 5250
+Connection ~ 1600 5250
+Wire Wire Line
+	1600 5250 1600 5300
+Wire Wire Line
+	3100 3550 3100 3600
+Wire Wire Line
+	3100 3900 3100 4000
+Wire Wire Line
+	3100 3600 4100 3600
+Wire Wire Line
+	4100 3600 4100 3650
+Connection ~ 3100 3600
+Wire Wire Line
+	3100 3600 3100 3700
+Wire Wire Line
+	3100 4000 4100 4000
+Wire Wire Line
+	4100 4000 4100 3950
+Connection ~ 3100 4000
+Wire Wire Line
+	3100 4000 3100 4050
 $EndSCHEMATC
